File: hardware/PCB-PHX-PALM-001.kicad_sch (KiCad schematic)
At the start: 2 parts, among them U101 NDP120-B0-CB-01, U201 PGA460TPWR

Commit message: Hardware Fix: Replace ultrasonic PGA460 chip with TI ADS1299 24-Bit sEMG AFE & Otto Bock 13E200 active electrode interface in KiCAD schematics, netlists, C firmware, and documentation
Parts:
- added J201: MyoBock_13E200_Quad, symbol OttoBock:13E200_Header
- U201: value PGA460TPWR -> ADS1299IPAG; symbol TI:PGA460 -> TI:ADS1299
Changed lines of the file:
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@@
     (company "Project Phoenix MedTech")
     (comment 1 "Indian Patent Application No. 202641077314")
-    (comment 2 "Syntiant NDP120 + PGA460 sEMG + MCP2518FD CAN-FD")
+    (comment 2 "Syntiant NDP120 + TI ADS1299 sEMG AFE + MCP2518FD CAN-FD")
   )
   (symbol (lib_id "Syntiant:NDP120") (at 100 100 0) (unit 1)
@@
     (property "Value" "NDP120-B0-CB-01" (at 100 110 0))
   )
-  (symbol (lib_id "TI:PGA460") (at 180 100 0) (unit 1)
+  (symbol (lib_id "TI:ADS1299") (at 180 100 0) (unit 1)
     (in_bom yes) (on_board yes) (fields_autoplaced yes)
     (property "Reference" "U201" (at 180 90 0))
-    (property "Value" "PGA460TPWR" (at 180 110 0))
+    (property "Value" "ADS1299IPAG" (at 180 110 0))
+  )
+  (symbol (lib_id "OttoBock:13E200_Header") (at 240 100 0) (unit 1)
+    (in_bom yes) (on_board yes) (fields_autoplaced yes)
+    (property "Reference" "J201" (at 240 90 0))
+    (property "Value" "MyoBock_13E200_Quad" (at 240 110 0))
   )
   (sheet_instances
